File: kimchi-camera-lid.sch (KiCad schematic (older format))
At the start: 21 parts, among them J1 DF40HC(3.5)-60DS, J2 DF40HC(3.5)-60DS, J3 DF40C-60DP, J4 DF40C-60DP, J5 Conn_01x15_MountingPin, J6 Conn_01x15_MountingPin, J7 Conn_01x22_MountingPin, J8 Conn_01x02, K1 KIMCHI_MICRO, U1 24C32

Commit message: Complete design for v1.0
Parts:
- D1: Mfgr (none) -> Nexperia; Mfgrpart (none) -> PMEG1020EH,115; Vendorpart (none) -> 1727-3849-1-ND
- J1, J2: Mfgr (none) -> Hirose; Mfgrpart (none) -> DF40HC(3.5)-60DS-0.4V(51); Vendorpart (none) -> H11917CT-ND
- J3, J4: symbol Connector_Generic:Conn_02x30_Counter_Clockwise -> Connector_Generic_MountingPin:Conn_02x30_Counter_Clockwise_MountingPin
- K1, L1, LOGO1: Populate (none) -> DNP
- U1: Mfgrpart (none) -> M24C32-FMC6TG; Part M24C32-FMC6TG -> (none)
Connections:
- net GND: now also J3.MP (MountPin), J4.MP (MountPin)
- net P2_42: now reaches J2.42 (Pin_42)
- net P2_42: now also J4.42 (Pin_42)
- net P2_54: now reaches J2.54 (Pin_54)
- net P2_54: now also J4.54 (Pin_54)
- net P2_58: now reaches J2.58 (Pin_58)
- net P2_58: now also J4.58 (Pin_58)
- net P1_11: now reaches J1.11 (Pin_11)
- net P1_11: now also J3.11 (Pin_11)
- net P1_51: now reaches J1.51 (Pin_51)
- net P1_51: now also J3.51 (Pin_51)
- no-connect marks 20 -> 10
Changed lines of the file:
@@
 F 3 "http://www.st.com/content/ccc/resource/technical/document/datasheet/80/4e/8c/54/f2/63/4c/4a/CD00001012.pdf/files/CD00001012.pdf/jcr:content/translations/en.CD00001012.pdf" H 11800 1700 50  0001 C CNN
 F 4 "ST" H 11800 1700 50  0001 C CNN "Mfgr"
-F 5 "M24C32-FMC6TG" H 11800 1700 50  0001 C CNN "Part"
+F 5 "" H 11800 1700 50  0001 C CNN "Part"
 F 6 "497-15757-1-ND" H 11800 1700 50  0001 C CNN "Vendorpart"
+F 7 "M24C32-FMC6TG" H 11800 1700 50  0001 C CNN "Mfgrpart"
 	1    11800 1700
 	1    0    0    -1
@@
 F 2 "Symbol:OSHW-Logo_5.7x6mm_SilkScreen" H 12000 10300 50  0001 C CNN
 F 3 "~" H 12000 10300 50  0001 C CNN
+F 4 "DNP" H 12000 10300 50  0001 C CNN "Populate"
 	1    12000 10300
 	1    0    0    -1
@@
 F 2 "kimchi_ulid:DF40HC(3.5)-60DS" H 5050 2850 50  0001 C CNN
 F 3 "~" H 5050 2850 50  0001 C CNN
+F 4 "Hirose" H 5050 2850 50  0001 C CNN "Mfgr"
+F 5 "DF40HC(3.5)-60DS-0.4V(51)" H 5050 2850 50  0001 C CNN "Mfgrpart"
+F 6 "H11917CT-ND" H 5050 2850 50  0001 C CNN "Vendorpart"
 	1    5050 2850
 	1    0    0    -1
@@
 	2250 2750 1200 2750
 $Comp
-L Connector_Generic:Conn_02x30_Counter_Clockwise J1
-U 1 1 5E5E1603
-P 2450 2850
-AR Path="/5E5E1603" Ref="J1"  Part="1"
-AR Path="/5E34BAA5/5E5E1603" Ref="J?"  Part="1"
-F 0 "J1" H 2500 4467 50  0000 C CNN
-F 1 "DF40HC(3.5)-60DS" H 2500 4376 50  0000 C CNN
-F 2 "kimchi_ulid:DF40HC(3.5)-60DS" H 2450 2850 50  0001 C CNN
-F 3 "~" H 2450 2850 50  0001 C CNN
-	1    2450 2850
-	1    0    0    -1
-$EndComp
-$Comp
 L power:PWR_FLAG #FLG0101
 U 1 1 5E5F10BC
@@
 Wire Wire Line
 	3300 2250 2750 2250
-NoConn ~ 2750 2350
 Text Notes 6300 3100 0    50   ~ 0
 0.9A max
-NoConn ~ 5350 2050
-NoConn ~ 5350 3250
-NoConn ~ 2250 2450
 Wire Wire Line
 	2250 2350 1200 2350
@@
 Text Notes 13450 850  0    50   ~ 0
 Recommend standoffs populated on lid\nMatch height of J1/J2 (typ. 3.5 mm)\nWürth WA-SMST 9774035943R (non-threaded)\nWürth WA-SMSI 9774035243R (threaded)
-NoConn ~ 5350 1650
 $Comp
 L kimchi_ulid:KIMCHI_MICRO K1
 U 1 1 60D1AF4A
-P 11050 10300
-F 0 "K1" H 11075 10346 50  0000 L CNN
-F 1 "KIMCHI_MICRO" H 11075 10255 50  0000 L CNN
-F 2 "kimchi_ulid:KIMCHI_MICRO" H 11050 10300 50  0001 C CNN
-F 3 "" H 11050 10300 50  0001 C CNN
-	1    11050 10300
-	1    0    0    -1
-$EndComp
-$Comp
-L Connector_Generic:Conn_02x30_Counter_Clockwise J4
+P 11100 10300
+F 0 "K1" H 11125 10346 50  0000 L CNN
+F 1 "KIMCHI_MICRO" H 11125 10255 50  0000 L CNN
+F 2 "kimchi_ulid:KIMCHI_MICRO" H 11100 10300 50  0001 C CNN
+F 3 "" H 11100 10300 50  0001 C CNN
+F 4 "DNP" H 11100 10300 50  0001 C CNN "Populate"
+	1    11100 10300
+	1    0    0    -1
+$EndComp
+$Comp
+L Connector_Generic_MountingPin:Conn_02x30_Counter_Clockwise_MountingPin J4
 U 1 1 60D90730
 P 5050 8000
@@
 	2250 7900 1200 7900
 $Comp
-L Connector_Generic:Conn_02x30_Counter_Clockwise J3
+L Connector_Generic_MountingPin:Conn_02x30_Counter_Clockwise_MountingPin J3
 U 1 1 60D907FA
 P 2450 8000
@@
 Wire Wire Line
 	3300 7400 2750 7400
-NoConn ~ 2750 7500
-NoConn ~ 5350 7200
-NoConn ~ 5350 8400
-NoConn ~ 2250 7600
 Wire Wire Line
 	2250 7500 1200 7500
@@
 	1200 7500 1200 7400
 Connection ~ 1200 7400
-NoConn ~ 5350 6800
 $Comp
 L Connector_Generic_MountingPin:Conn_01x15_MountingPin J5
@@
 F 2 "Diode_SMD:D_SOD-123F" H 12450 2975 50  0001 C CNN
 F 3 "https://assets.nexperia.com/documents/data-sheet/PMEG1020EH_EJ.pdf" H 12450 3150 50  0001 C CNN
+F 4 "1727-3849-1-ND" H 12450 3150 50  0001 C CNN "Vendorpart"
+F 5 "Nexperia" H 12450 3150 50  0001 C CNN "Mfgr"
+F 6 "PMEG1020EH,115" H 12450 3150 50  0001 C CNN "Mfgrpart"
 	1    12450 3150
 	1    0    0    -1
@@
 F 2 "kimchi_ulid:gg-4x4" H 10550 10300 50  0001 C CNN
 F 3 "" H 10550 10300 50  0001 C CNN
+F 4 "DNP" H 10550 10300 50  0001 C CNN "Populate"
 	1    10550 10300
 	1    0    0    -1
 $EndComp
+Text Label 2250 2450 2    50   ~ 0
+P1_11
+Text Label 2250 7600 2    50   ~ 0
+P1_11
+Text Label 5350 1650 0    50   ~ 0
+P2_58
+Text Label 5350 6800 0    50   ~ 0
+P2_58
+Text Label 5350 7200 0    50   ~ 0
+P2_54
+Text Label 5350 2050 0    50   ~ 0
+P2_54
+Text Label 5350 3250 0    50   ~ 0
+P2_42
+Text Label 5350 8400 0    50   ~ 0
+P2_42
+Text Label 2750 7500 0    50   ~ 0
+P1_51
+Text Label 2750 2350 0    50   ~ 0
+P1_51
+$Comp
+L Connector_Generic:Conn_02x30_Counter_Clockwise J1
+U 1 1 5E5E1603
+P 2450 2850
+AR Path="/5E5E1603" Ref="J1"  Part="1"
+AR Path="/5E34BAA5/5E5E1603" Ref="J?"  Part="1"
+F 0 "J1" H 2500 4467 50  0000 C CNN
+F 1 "DF40HC(3.5)-60DS" H 2500 4376 50  0000 C CNN
+F 2 "kimchi_ulid:DF40HC(3.5)-60DS" H 2450 2850 50  0001 C CNN
+F 3 "~" H 2450 2850 50  0001 C CNN
+F 4 "H11917CT-ND" H 2450 2850 50  0001 C CNN "Vendorpart"
+F 5 "Hirose" H 2450 2850 50  0001 C CNN "Mfgr"
+F 6 "DF40HC(3.5)-60DS-0.4V(51)" H 2450 2850 50  0001 C CNN "Mfgrpart"
+	1    2450 2850
+	1    0    0    -1
+$EndComp
+$Comp
+L power:GND #PWR0133
+U 1 1 6110C964
+P 2500 9700
+F 0 "#PWR0133" H 2500 9450 50  0001 C CNN
+F 1 "GND" H 2505 9527 50  0000 C CNN
+F 2 "" H 2500 9700 50  0001 C CNN
+F 3 "" H 2500 9700 50  0001 C CNN
+	1    2500 9700
+	1    0    0    -1
+$EndComp
+$Comp
+L power:GND #PWR0134
+U 1 1 6110CDDD
+P 5100 9700
+F 0 "#PWR0134" H 5100 9450 50  0001 C CNN
+F 1 "GND" H 5105 9527 50  0000 C CNN
+F 2 "" H 5100 9700 50  0001 C CNN
+F 3 "" H 5100 9700 50  0001 C CNN
+	1    5100 9700
+	1    0    0    -1
+$EndComp
